Commit message: Fully working 6 dof robot in gazebo with ros2_control

File: ra6dof_description/gazebo/gazebo_sim_ros2_control.urdf.xacro (robot description, xacro)
@@ -1,9 +1,9 @@
 <?xml version="1.0" ?>
 <robot xmlns:xacro="http://wiki.ros.org/xacro">
-    <xacro:macro name="load_gazebo_sim_ros2_control_plugin" params="robot_name use_gazebo">
+    <xacro:macro name="load_gazebo_sim_ros2_control_plugin" params="use_gazebo">
         <xacro:if value="${use_gazebo}">
             <gazebo>
                 <plugin filename="gz_ros2_control-system" name="gz_ros2_control::GazeboSimROS2ControlPlugin">
-                    <parameters>$(find mycobot_moveit_config)/config/${robot_name}/ros2_controllers.yaml</parameters>
+                    <parameters>$(find ra6dof_controller)/config/mycobot_280_controllers.yaml</parameters>
                     <ros>
                         <remapping>/controller_manager/robot_description:=/robot_description</remapping>

File: ra6dof_description/ros2_control/mycobot_280_ros2_control.urdf.xacro (robot description, xacro)
@@ -1,5 +1,5 @@
 <?xml version="1.0" ?>
 <robot xmlns:xacro="http://wiki.ros.org/xacro">
-    <xacro:macro name="mycobot_ros2_control" params="prefix flange_link use_gazebo">
+    <xacro:macro name="mycobot_ros2_control" params="prefix use_gazebo">
         <ros2_control name="RobotSystem" type="system">
             <hardware>
@@ -8,5 +8,5 @@
                 </xacro:if>
             </hardware>
-            <joint name="${prefix}link1_to_${prefix}link2">
+            <joint name="link1_to_link2">
                 <command_interface name="position">
                     <param name="min">-2.879793</param>
@@ -15,5 +15,5 @@
                 <state_interface name="position"/>
             </joint>
-            <joint name="${prefix}link2_to_${prefix}link3">
+            <joint name="link2_to_link3">
                 <command_interface name="position">
                     <param name="min">-2.879793</param>
@@ -22,5 +22,5 @@
                 <state_interface name="position"/>
             </joint>
-            <joint name="${prefix}link3_to_${prefix}link4">
+            <joint name="link3_to_link4">
                 <command_interface name="position">
                     <param name="min">-2.879793</param>
@@ -29,5 +29,5 @@
                 <state_interface name="position"/>
             </joint>
-            <joint name="${prefix}link4_to_${prefix}link5">
+            <joint name="link4_to_link5">
                 <command_interface name="position">
                     <param name="min">-2.879793</param>
@@ -36,5 +36,5 @@
                 <state_interface name="position"/>
             </joint>
-            <joint name="${prefix}link5_to_${prefix}link6">
+            <joint name="link5_to_link6">
                 <command_interface name="position">
                     <param name="min">-2.879793</param>
@@ -43,5 +43,5 @@
                 <state_interface name="position"/>
             </joint>
-            <joint name="${prefix}link6_to_${prefix}${flange_link}">
+            <joint name="link6_to_flange">
                 <command_interface name="position">
                     <param name="min">-3.05</param>
@@ -50,5 +50,5 @@
                 <state_interface name="position"/>
             </joint>
-            <joint name="${prefix}gripper_controller">
+            <joint name="gripper_controller">
                 <command_interface name="position">
                     <param name="min">-0.7</param>

File: ra6dof_description/urdf/end_effector/adaptive_gripper.urdf.xacro (robot description, xacro)
@@ -137,5 +137,5 @@
       </collision>
     </link>
-    <joint name="${prefix}gripper_controller" type="revolute">
+    <joint name="gripper_controller" type="revolute">
       <axis xyz="0 0 1"/>
       <limit effort="${joint_effort}" lower="-0.7" upper="0.15" velocity="${joint_velocity}"/>
@@ -151,5 +151,5 @@
       <child link="${prefix}gripper_left2"/>
       <origin xyz="-0.005 0.027 0" rpy="0 0 0"/>
-      <mimic joint="${prefix}gripper_controller" multiplier="1.0" offset="0"/>
+      <mimic joint="gripper_controller" multiplier="1.0" offset="0"/>
       <dynamics damping="${joint_damping}" friction="${joint_friction}"/>
     </joint>
@@ -160,5 +160,5 @@
       <child link="${prefix}gripper_left1"/>
       <origin xyz="-0.027 0.016 0" rpy="0 0 0"/>
-      <mimic joint="${prefix}gripper_controller" multiplier="-1.0" offset="0"/>
+      <mimic joint="gripper_controller" multiplier="-1.0" offset="0"/>
       <dynamics damping="${joint_damping}" friction="${joint_friction}"/>
     </joint>
@@ -169,5 +169,5 @@
       <child link="${prefix}gripper_right3"/>
       <origin xyz="0.012 0.005 0" rpy="0 0 0"/>
-      <mimic joint="${prefix}gripper_controller" multiplier="-1.0" offset="0"/>
+      <mimic joint="gripper_controller" multiplier="-1.0" offset="0"/>
       <dynamics damping="${joint_damping}" friction="${joint_friction}"/>
     </joint>
@@ -178,5 +178,5 @@
       <child link="${prefix}gripper_right2"/>
       <origin xyz="0.005 0.027 0" rpy="0 0 0"/>
-      <mimic joint="${prefix}gripper_controller" multiplier="-1.0" offset="0"/>
+      <mimic joint="gripper_controller" multiplier="-1.0" offset="0"/>
       <dynamics damping="${joint_damping}" friction="${joint_friction}"/>
     </joint>
@@ -187,5 +187,5 @@
       <child link="${prefix}gripper_right1"/>
       <origin xyz="0.027 0.016 0" rpy="0 0 0"/>
-      <mimic joint="${prefix}gripper_controller" multiplier="1.0" offset="0"/>
+      <mimic joint="gripper_controller" multiplier="1.0" offset="0"/>
       <dynamics damping="${joint_damping}" friction="${joint_friction}"/>
     </joint>

File: ra6dof_description/urdf/mycobot_280.urdf.xacro (robot description, xacro)
@@ -9,5 +9,5 @@
     <xacro:arg name="prefix" default=""/>
     <xacro:arg name="use_camera" default="false"/>
-    <xacro:arg name="use_gazebo" default="false"/>
+    <xacro:arg name="use_gazebo" default="true"/>
     <xacro:arg name="use_gripper" default="true"/>
     <xacro:if value="$(arg add_world)">
@@ -21,10 +21,10 @@
     <xacro:property name="current_base" value="$(arg base_type)"/>
     <xacro:if value="${current_base == 'g_shape'}">
-        <xacro:include filename="g_shape_base_v2_0.urdf.xacro"/>
+        <xacro:include filename="robot/g_shape_base_v2_0.urdf.xacro"/>
         <xacro:g_shape_base
             base_link="$(arg base_link)"
             prefix="$(arg prefix)"/>
     </xacro:if>
-    <xacro:include filename="mycobot_280_arm.urdf.xacro"/>
+    <xacro:include filename="robot/mycobot_280_arm.urdf.xacro"/>
     <xacro:mycobot_280_arm
       base_link="$(arg base_link)"
@@ -36,5 +36,5 @@
         <xacro:property name="current_gripper" value="$(arg gripper_type)"/>
         <xacro:if value="${current_gripper == 'adaptive_gripper'}">
-            <xacro:include filename="adaptive_gripper.urdf.xacro"/>
+            <xacro:include filename="end_effector/adaptive_gripper.urdf.xacro"/>
             <xacro:adaptive_gripper
                 parent="$(arg flange_link)"
@@ -44,15 +44,11 @@
         </xacro:if>
     </xacro:if>
-<!--
-    <xacro:include filename="gazebo_sim_ros2_control.urdf.xacro" />
+    <xacro:include filename="$(find ra6dof_description)/gazebo/gazebo_sim_ros2_control.urdf.xacro" />
     <xacro:load_gazebo_sim_ros2_control_plugin
-      robot_name="$(arg robot_name)"
       use_gazebo="$(arg use_gazebo)"/>
-    <xacro:include filename="mycobot_280_ros2_control.urdf.xacro" />
+    <xacro:include filename="$(find ra6dof_description)/ros2_control/mycobot_280_ros2_control.urdf.xacro" />
     <xacro:mycobot_ros2_control
       prefix="$(arg prefix)"
-      flange_link="$(arg flange_link)"
       use_gazebo="$(arg use_gazebo)"/>
-    <xacro:include filename="intel_rgbd_cam_d435.urdf.xacro"/>
- -->
+    <!-- <xacro:include filename="sensors/intel_rgbd_cam_d435.urdf.xacro"/> -->
 </robot>

File: ra6dof_description/urdf/robot/mycobot_280_arm.urdf.xacro (robot description, xacro)
@@ -144,5 +144,5 @@
       <xacro:insert_block name="origin"/>
     </joint>
-    <joint name="${prefix}link1_to_${prefix}link2" type="revolute">
+    <joint name="link1_to_link2" type="revolute">
       <axis xyz="0 0 1"/>
       <limit effort="${joint_effort}" lower="-2.879793" upper="2.879793" velocity="${joint_velocity}"/>
@@ -152,5 +152,5 @@
       <dynamics damping="${joint_damping}" friction="${joint_friction}"/>
     </joint>
-    <joint name="${prefix}link2_to_${prefix}link3" type="revolute">
+    <joint name="link2_to_link3" type="revolute">
       <axis xyz="0 0 1"/>
       <limit effort="${joint_effort}" lower="-2.879793" upper="2.879793" velocity="${joint_velocity}"/>
@@ -160,5 +160,5 @@
       <dynamics damping="${joint_damping}" friction="${joint_friction}"/>
     </joint>
-    <joint name="${prefix}link3_to_${prefix}link4" type="revolute">
+    <joint name="link3_to_link4" type="revolute">
       <axis xyz="0 0 1"/>
       <limit effort="${joint_effort}" lower="-2.879793" upper="2.879793" velocity="${joint_velocity}"/>
@@ -168,5 +168,5 @@
       <dynamics damping="${joint_damping}" friction="${joint_friction}"/>
     </joint>
-    <joint name="${prefix}link4_to_${prefix}link5" type="revolute">
+    <joint name="link4_to_link5" type="revolute">
       <axis xyz="0 0 1"/>
       <limit effort="${joint_effort}" lower="-2.879793" upper="2.879793" velocity="${joint_velocity}"/>
@@ -176,5 +176,5 @@
       <dynamics damping="${joint_damping}" friction="${joint_friction}"/>
     </joint>
-    <joint name="${prefix}link5_to_${prefix}link6" type="revolute">
+    <joint name="link5_to_link6" type="revolute">
       <axis xyz="0 0 1"/>
       <limit effort="${joint_effort}" lower="-2.879793" upper="2.879793" velocity="${joint_velocity}"/>
@@ -184,5 +184,5 @@
       <dynamics damping="${joint_damping}" friction="${joint_friction}"/>
     </joint>
-    <joint name="${prefix}link6_to_${prefix}${flange_link}" type="revolute">
+    <joint name="link6_to_flange" type="revolute">
       <axis xyz="0 0 1"/>
       <limit effort="${joint_effort}" lower="-3.05" upper="3.05" velocity="${joint_velocity}"/>
